File: hardware/halogen-led.sch (EAGLE design)
At the start: 33 parts

Commit message: rc2
Parts:
- C1: value 10u -> 25u
- C2: value 1u -> 25u
Other:
- note added: "Input + Rectifier"
- note added: "Main LEDs"
- note added: "Secondary LEDs"
- moved on the sheet: B1, C1, C2, C3, C4, D1, D2, D3, D4, D5, D6, D7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

Commit message: hw: changed some values
Parts:
- C1, C2: value 25u -> DNP
- C3, C4: value 10u -> DNP
- R1: value Rshunt -> 22 (blue), 10 (others)
- R2, R3: value Rshunt -> 10
- R4, R5, R6: value Req -> 0
Other:
- moved on the sheet: C4
Changed lines of the file:
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@@
 <part name="JP1" library="SparkFun-Connectors" deviceset="M01" device="PTH"/>
 <part name="JP2" library="SparkFun-Connectors" deviceset="M01" device="PTH"/>
-<part name="C1" library="rcl" deviceset="C-EU" device="C1206" value="25u"/>
+<part name="C1" library="rcl" deviceset="C-EU" device="C1206" value="DNP"/>
 <part name="P+1" library="supply1" deviceset="VCC" device=""/>
 <part name="LED1" library="led" deviceset="LED" device="CHIPLED_0805"/>
-<part name="C2" library="rcl" deviceset="C-EU" device="C1206" value="25u"/>
+<part name="C2" library="rcl" deviceset="C-EU" device="C1206" value="DNP"/>
 <part name="GND2" library="supply1" deviceset="GND" device=""/>
 <part name="GND3" library="supply1" deviceset="GND" device=""/>
 <part name="IC1" library="SparkFun-PowerIC" deviceset="V_REG_LM1117" device="SOT223"/>
 <part name="P+2" library="supply1" deviceset="VCC" device=""/>
-<part name="R2" library="rcl" deviceset="R-EU_" device="R1206" value="Rshunt"/>
+<part name="R2" library="rcl" deviceset="R-EU_" device="R1206" value="10"/>
 <part name="B1" library="rectifier" deviceset="B*S" device="" technology="1"/>
 <part name="GND1" library="supply1" deviceset="GND" device=""/>
 <part name="IC2" library="SparkFun-PowerIC" deviceset="V_REG_LM1117" device="SOT223"/>
-<part name="R1" library="rcl" deviceset="R-EU_" device="R1206" value="Rshunt"/>
+<part name="R1" library="rcl" deviceset="R-EU_" device="R1206" value="22 (blue), 10 (others)"/>
 <part name="P+3" library="supply1" deviceset="VCC" device=""/>
 <part name="LED2" library="led" deviceset="LED" device="CHIPLED_0805"/>
@@
 <part name="GND5" library="supply1" deviceset="GND" device=""/>
 <part name="GND6" library="supply1" deviceset="GND" device=""/>
-<part name="C3" library="rcl" deviceset="C-EU" device="C0805" value="10u"/>
+<part name="C3" library="rcl" deviceset="C-EU" device="C0805" value="DNP"/>
 <part name="GND7" library="supply1" deviceset="GND" device=""/>
-<part name="C4" library="rcl" deviceset="C-EU" device="C0805" value="10u"/>
+<part name="C4" library="rcl" deviceset="C-EU" device="C0805" value="DNP"/>
 <part name="GND8" library="supply1" deviceset="GND" device=""/>
 <part name="D7" library="balto" deviceset="LED_XH-G" device=""/>
@@
 <part name="D9" library="balto" deviceset="LED_XH-G" device=""/>
 <part name="GND9" library="supply1" deviceset="GND" device=""/>
-<part name="R3" library="rcl" deviceset="R-EU_" device="R1206" value="Rshunt"/>
+<part name="R3" library="rcl" deviceset="R-EU_" device="R1206" value="10"/>
 <part name="LED6" library="led" deviceset="LED" device="CHIPLED_0805"/>
 <part name="LED7" library="led" deviceset="LED" device="CHIPLED_0805"/>
@@
 <part name="LED9" library="led" deviceset="LED" device="CHIPLED_0805"/>
 <part name="GND10" library="supply1" deviceset="GND" device=""/>
-<part name="R4" library="rcl" deviceset="R-EU_" device="R0805" value="Req"/>
-<part name="R5" library="rcl" deviceset="R-EU_" device="R0805" value="Req"/>
-<part name="R6" library="rcl" deviceset="R-EU_" device="R0805" value="Req"/>
+<part name="R4" library="rcl" deviceset="R-EU_" device="R0805" value="0"/>
+<part name="R5" library="rcl" deviceset="R-EU_" device="R0805" value="0"/>
+<part name="R6" library="rcl" deviceset="R-EU_" device="R0805" value="0"/>
 <part name="SJ1" library="SparkFun-Passives" deviceset="SOLDERJUMPER" device="NC2"/>
 </parts>
@@
 <instance part="C3" gate="G$1" x="99.06" y="142.24"/>
 <instance part="GND7" gate="1" x="99.06" y="132.08"/>
-<instance part="C4" gate="G$1" x="185.42" y="142.24"/>
-<instance part="GND8" gate="1" x="185.42" y="132.08"/>
+<instance part="C4" gate="G$1" x="203.2" y="142.24"/>
+<instance part="GND8" gate="1" x="203.2" y="132.08"/>
 <instance part="D7" gate="G$1" x="111.76" y="106.68" smashed="yes">
 <attribute name="NAME" x="114.808" y="105.664" size="1.778" layer="95"/>
@@
 <pinref part="GND8" gate="1" pin="GND"/>
 <pinref part="C4" gate="G$1" pin="2"/>
-<wire x1="185.42" y1="134.62" x2="185.42" y2="137.16" width="0.1524" layer="91"/>
+<wire x1="203.2" y1="134.62" x2="203.2" y2="137.16" width="0.1524" layer="91"/>
 </segment>
 <segment>
@@
 <segment>
 <pinref part="C4" gate="G$1" pin="1"/>
-<wire x1="185.42" y1="149.86" x2="185.42" y2="144.78" width="0.1524" layer="91"/>
+<wire x1="203.2" y1="149.86" x2="203.2" y2="144.78" width="0.1524" layer="91"/>
 <pinref part="IC2" gate="G$1" pin="OUT@1"/>
 <pinref part="R1" gate="G$1" pin="2"/>
@@
 <wire x1="165.1" y1="149.86" x2="165.1" y2="147.32" width="0.1524" layer="91"/>
 <junction x="165.1" y="147.32"/>
-<wire x1="185.42" y1="149.86" x2="165.1" y2="149.86" width="0.1524" layer="91"/>
+<wire x1="203.2" y1="149.86" x2="165.1" y2="149.86" width="0.1524" layer="91"/>
 <junction x="165.1" y="149.86"/>
 </segment>
